Commit message: 新版本-lsh-sfdevelop

File: resources/robots/wl/urdf/wl.urdf (robot description, URDF)
Before this commit: robot wl, 7 links, 6 joints
Joints:
- joint l_wheel_Joint: limit effort=5 velocity=1000 -> effort=5 velocity=300
- joint lf0_Joint: limit lower=-0.3363 upper=1.3479 effort=30 velocity=1000 -> lower=-0.3363 upper=1.3479 effort=30 velocity=30
- joint lf1_Joint: limit lower=-1.0 upper=1.25 effort=30 velocity=1000 -> lower=-1.0 upper=1.25 effort=30 velocity=30
- joint r_wheel_Joint: limit effort=5 velocity=1000 -> effort=5 velocity=300
- joint rf0_Joint: limit lower=-1.3479 upper=0.3363 effort=30 velocity=1000 -> lower=-1.3479 upper=0.3363 effort=30 velocity=30
- joint rf1_Joint: limit lower=-1.25 upper=1.0 effort=30 velocity=1000 -> lower=-1.25 upper=1.0 effort=30 velocity=30
