Commit message: update

File: resources/robots/sf/urdf/sfrviz.urdf (robot description, URDF)
Before this commit: robot sf, 7 links, 6 joints
Joints:
- joint LW_joint: limit lower=-1000000 upper=1000000 effort=0.25 velocity=100 -> lower=-1000000 upper=1000000 effort=0.1 velocity=100
- joint RW_joint: limit lower=-1000000 upper=1000000 effort=0.25 velocity=100 -> lower=-1000000 upper=1000000 effort=0.1 velocity=100
